Commit message: working network and skills.

File: models/arena.xacro (robot description, xacro)
@@ -18,5 +18,5 @@
 	</material>
 	<material name="black">
-		<color rgba="0 0 0 1"/>
+		<color rgba="1 0 1 1"/>
 	</material>
 	<material name="green">
@@ -51,21 +51,4 @@
 		</contact>
 	</link>
-	<link name="start_pad">
-		<inertial>
-			<mass value="0.1"/>
-			<inertia ixx="0.001" ixy="0" ixz="0" iyy="0.001" iyz="0" izz="0.001"/>
-		</inertial>
-		<visual>
-			<geometry>
-				<box size="0.1 0.1 0.001"/>
-			</geometry>
-			<material name="white"/>
-		</visual>
-	</link>
-	<joint name="start_joint" type="fixed">
-		<parent link="floor"/>
-		<child link="start_pad"/>
-		<origin xyz="${-(floor_x * 0.375)} 0 0.001"/>
-	</joint>
 	<link name="end_pad">
 		<inertial>
@@ -83,5 +66,5 @@
 		<parent link="floor"/>
 		<child link="end_pad"/>
-		<origin xyz="${floor_x*0.375} 0 0.001"/>
+		<origin xyz="${floor_x*0.375} ${floor_y * 0.375} 0.001"/>
 	</joint>
 	<link name="walls">

File: models/urdfs/arena.urdf (robot description, URDF)
Before this commit: robot arena, 6 links, 5 joints
Links:
- removed link start_pad
Joints:
- removed joint start_joint
- joint end_joint: origin xyz=0.375 0 0.001 -> xyz=0.375 0.375 0.001

Commit message: koniec dnia 28.08

File: models/arena.xacro (robot description, xacro)
@@ -18,5 +18,5 @@
 	</material>
 	<material name="black">
-		<color rgba="1 0 1 1"/>
+		<color rgba="0 0 0 1"/>
 	</material>
 	<material name="green">
@@ -24,5 +24,5 @@
 	</material>
 	<material name="blue">
-		<color rgba="0.4 0.6 1 1"/>
+		<color rgba="0.5 0.5 1 1"/>
 	</material>
 	<material name="red">
@@ -51,5 +51,5 @@
 		</contact>
 	</link>
-	<link name="end_pad">
+	<link name="end_column">
 		<inertial>
 			<mass value="0.1"/>
@@ -57,14 +57,21 @@
 		</inertial>
 		<visual>
-			<geometry>
-				<box size="0.1 0.1 0.001"/>
+			<origin xyz="0 0 ${wall_height/2}"/>
+			<geometry>
+				<box size="0.1 0.01 ${wall_height}"/>
 			</geometry>
 			<material name="blue"/>
 		</visual>
+		<collision>
+			<origin xyz="0 0 ${wall_height/2}"/>
+			<geometry>
+				<box size="0.1 0.01 ${wall_height}"/>
+			</geometry>
+		</collision>
 	</link>
 	<joint name="end_joint" type="fixed">
 		<parent link="floor"/>
-		<child link="end_pad"/>
-		<origin xyz="${floor_x*0.375} ${floor_y * 0.375} 0.001"/>
+		<child link="end_column"/>
+		<origin xyz="${floor_x*0.375} ${floor_y * 0.45} 0"/>
 	</joint>
 	<link name="walls">

File: models/urdfs/arena.urdf (robot description, URDF)
Before this commit: robot arena, 5 links, 4 joints
Links:
- removed link end_pad
- added link end_column, mass 0.1; collision box size=0.1 0.01 0.2; visual box size=0.1 0.01 0.2
Joints:
- joint end_joint: child end_pad -> end_column; origin xyz=0.375 0.375 0.001 -> xyz=0.375 0.45 0

Commit message: working linear skills (finally)

File: models/arena.xacro (robot description, xacro)
@@ -18,5 +18,5 @@
 	</material>
 	<material name="black">
-		<color rgba="0 0 0 1"/>
+		<color rgba="0.2 0.2 0.2 1"/>
 	</material>
 	<material name="green">
@@ -202,5 +202,5 @@
 		<axis xyz="0 0 1"/>
 		<limit effort="100" lower="-1.57" upper="1.57" velocity="25"/>
-		<dynamics damping="0.01" friction="${door_friction}"/>
+		<dynamics damping="0.05" friction="${door_friction}" spring_stiffness="0.02" spring_reference="0"/>
 	</joint>
 </robot>

File: models/epuck2.xacro (robot description, xacro)
@@ -18,7 +18,7 @@
 	    </collision>
 	    <inertial>
-		    <mass value="0.1"/>
-		    <origin xyz="0 0 -0.02" rpy="0 0 0"/>
-		    <inertia ixx="0.005" ixy="0" ixz="0" iyy="0.005" iyz="0" izz="0.05"/>
+		    <mass value="0.2"/>
+		    <origin xyz="0 0 -0.035" rpy="0 0 0"/>
+			<inertia ixx="0.0001" ixy="0" ixz="0" iyy="0.0001" iyz="0" izz="0.00012"/>
 	    </inertial>
 	    <contact>
@@ -41,5 +41,5 @@
     </inertial>
 	<contact>
-		<lateral_friction value="10.0"/>
+		<lateral_friction value="1.0"/>
 	</contact>
   </link>
@@ -65,5 +65,5 @@
     </inertial>
 	<contact>
-		<lateral_friction value="10.0"/>
+		<lateral_friction value="1.0"/>
 	</contact>
   </link>
@@ -74,9 +74,36 @@
     <axis xyz="0 1 0"/>
   </joint>
+<!-- INVISIBLE BUMPER RING -->
+<!-- Placed low and made slightly wider than the base to bump walls first. -->
+<link name="bumper_ring">
+	<collision>s
+		<geometry>
+			<!-- Slightly wider than the 0.035 base, very thin -->
+			<cylinder length="0.005" radius="0.037"/>
+		</geometry>
+	</collision>
+	<inertial>
+		<mass value="0.001"/>
+		<inertia ixx="0.0000001" ixy="0" ixz="0" iyy="0.0000001" iyz="0" izz="0.0000001"/>
+	</inertial>
+	<contact>
+		<!-- Zero friction ensures it slides on walls instead of climbing -->
+		<lateral_friction value="0.0"/>
+	</contact>
+</link>
+<joint name="bumper_ring_joint" type="fixed">
+	<parent link="base_link"/>
+	<child link="bumper_ring"/>
+	<!-- Z = -0.035 - CoM -->
+	<origin xyz="0 0 -0.03" rpy="0 0 0"/>
+</joint>
+<!-- END INVISIBLE BUMPER RING -->
   <link name="caster_front">
+	  <!--
     <visual>
       <geometry><sphere radius="0.005"/></geometry>
       <material name="light_grey"/>
     </visual>
+	-->
     <collision>
       <geometry><sphere radius="0.005"/></geometry>
@@ -98,8 +125,10 @@
   </joint>
   <link name="caster_back">
+	<!--
     <visual>
       <geometry><sphere radius="0.005"/></geometry>
       <material name="light_grey"/>
     </visual>
+	-->
     <collision>
       <geometry><sphere radius="0.005"/></geometry>
@@ -120,9 +149,30 @@
     <origin xyz="-0.02 0 -0.03" rpy="0 0 0"/>
   </joint>
+	<!-- KAMERA-->
+	<link name="camera_link">
+		<!--
+		<visual>
+			<geometry>
+				<box size="0.002 0.005 0.005"/>
+			</geometry>
+			<material name="red"/>
+		</visual>
+		-->
+		<inertial>
+			<mass value="0.0"/>
+			<inertia ixx="0" ixy="0" ixz="0" iyy="0" iyz="0" izz="0"/>
+		</inertial>
+	</link>
+	<joint name="camera_joint" type="fixed">
+		<parent link="base_link"/>
+		<child link="camera_link"/>
+		<!-- x=0.036 (przed oczami), y=0 (środek), z=0.015 (wysokość oczu) -->
+		<origin xyz="0.02 0.0 0.015" rpy="0 0 0"/>
+	</joint>
 	<!-- OCZY -->
     <link name="eye_left">
 		<inertial>
-			<mass value="0.001"/>
-			<inertia ixx="0.0000001" ixy="0" ixz="0" iyy="0.0000001" iyz="0" izz="0.0000001"/>
+			<mass value="0.00001"/>
+			<inertia ixx="0.000000001" ixy="0" ixz="0" iyy="0.000000001" iyz="0" izz="0.000000001"/>
 		</inertial>
 	    <visual>
@@ -143,6 +193,6 @@
     <link name="eye_right">
 		<inertial>
-			<mass value="0.001"/>
-			<inertia ixx="0.0000001" ixy="0" ixz="0" iyy="0.0000001" iyz="0" izz="0.0000001"/>
+			<mass value="0.00001"/>
+			<inertia ixx="0.000000001" ixy="0" ixz="0" iyy="0.000000001" iyz="0" izz="0.000000001"/>
 		</inertial>
 	    <visual>

File: models/urdfs/epuck2.urdf (robot description, URDF)
Before this commit: robot epuck2, 7 links, 6 joints
Links:
- added link bumper_ring, mass 0.001; collision cylinder length=0.005 radius=0.037
- added link camera_link, mass 0.0
- link base_link: mass 0.1 -> 0.2
- link caster_back: geometry collision sphere radius=0.005
- link caster_front: geometry collision sphere radius=0.005
- link eye_left: mass 0.001 -> 0.00001
- link eye_right: mass 0.001 -> 0.00001
Joints:
- added joint bumper_ring_joint: type fixed, parent base_link, child bumper_ring, origin xyz=0 0 -0.03 rpy=0 0 0
- added joint camera_joint: type fixed, parent base_link, child camera_link, origin xyz=0.02 0.0 0.015 rpy=0 0 0
