Commit message: new result folder and more visualisations; new way of calculating local_radius

File: models/arena_color.xacro (robot description, xacro)
@@ -35,20 +35,5 @@
 			<inertia ixx="0" ixy="0" ixz="0" iyy="0" iyz="0" izz="0"/>
 		</inertial>
-		<!-- Left Room Visual -->
-		<visual>
-			<origin xyz="-${floor_x/4} 0 -0.01"/>
-			<geometry>
-				<box size="${floor_x/2} ${floor_y} 0.02"/>
-			</geometry>
-			<material name="floor_left"/>
-		</visual>
-		<!-- Right Room Visual -->
-		<visual>
-			<origin xyz="${floor_x/4} 0 -0.01"/>
-			<geometry>
-				<box size="${floor_x/2} ${floor_y} 0.02"/>
-			</geometry>
-			<material name="floor_right"/>
-		</visual>
+		<!-- Unified collision and physics remain here -->
 		<collision>
 			<origin xyz="0 0 -0.01"/>
@@ -61,4 +46,40 @@
 		</contact>
 	</link>
+	<!-- Left Room Visual Link -->
+	<link name="floor_left_visual">
+		<visual>
+			<origin xyz="-${floor_x/4} 0 -0.009"/>
+			<geometry>
+				<box size="${floor_x/2} ${floor_y} 0.02"/>
+			</geometry>
+			<material name="floor_left"/>
+		</visual>
+		<inertial>
+			<mass value="0"/>
+			<inertia ixx="0" ixy="0" ixz="0" iyy="0" iyz="0" izz="0"/>
+		</inertial>
+	</link>
+	<joint name="floor_left_joint" type="fixed">
+		<parent link="floor"/>
+		<child link="floor_left_visual"/>
+	</joint>
+	<!-- Right Room Visual Link -->
+	<link name="floor_right_visual">
+		<visual>
+			<origin xyz="${floor_x/4} 0 -0.009"/>
+			<geometry>
+				<box size="${floor_x/2} ${floor_y} 0.02"/>
+			</geometry>
+			<material name="floor_right"/>
+		</visual>
+		<inertial>
+			<mass value="0"/>
+			<inertia ixx="0" ixy="0" ixz="0" iyy="0" iyz="0" izz="0"/>
+		</inertial>
+	</link>
+	<joint name="floor_right_joint" type="fixed">
+		<parent link="floor"/>
+		<child link="floor_right_visual"/>
+	</joint>
 	<link name="end_column">
 		<inertial>

File: models/urdfs/arena_color.urdf (robot description, URDF)
Before this commit: robot arena, 5 links, 4 joints
Links:
- added link floor_left_visual, mass 0; visual box size=0.5 1.0 0.02
- added link floor_right_visual, mass 0; visual box size=0.5 1.0 0.02
- link floor: geometry collision box size=1.0 1.0 0.02
Joints:
- added joint floor_left_joint: type fixed, parent floor, child floor_left_visual
- added joint floor_right_joint: type fixed, parent floor, child floor_right_visual
